File: kicad-smd/data-io.kicad_sch (KiCad schematic)
At the start: 45 parts, among them SW1 SW_DIP_x08

Commit message: smd schema text fixes
Other:
- note added: "3x push buttons with pull-up. Negative logic: press = 0."
- note added: "8x 0402 LED for digital output signals."
- note added: "8x DIP switches set GND, switch "off" uses internal pull-ups for '1' state."
- note added: "Input: DIP Switches"
- note removed: "2x push buttons with pull-up. Negative logic: press = 0."
- note removed: "4x 3mm LED for digital output signals."
- note removed: "4x slide switches set GND / +2V5 level signals."
- note removed: "Input: Slide Switches"
Changed lines of the file:
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@@
     (effects (font (size 2 2)) (justify left bottom))
   )
-  (text "2x push buttons with pull-up. Negative logic: press = 0."
+  (text "3x push buttons with pull-up. Negative logic: press = 0."
     (at 19.05 25.4 0)
     (effects (font (size 1.27 1.27)) (justify left bottom))
@@
     (effects (font (size 2.54 2.54) (thickness 0.4) bold) (justify left bottom))
   )
-  (text "4x slide switches set GND / +2V5 level signals." (at 20.32 87.63 0)
+  (text "8x DIP switches set GND, switch \"off\" uses internal pull-ups for '1' state."
+    (at 20.32 87.63 0)
     (effects (font (size 1.27 1.27)) (justify left bottom))
   )
-  (text "Input: Slide Switches" (at 20.32 85.09 0)
+  (text "Input: DIP Switches" (at 20.32 85.09 0)
     (effects (font (size 2.54 2.54) (thickness 0.4) bold) (justify left bottom))
   )
-  (text "4x 3mm LED for digital output signals." (at 100.33 87.63 0)
+  (text "8x 0402 LED for digital output signals." (at 100.33 87.63 0)
     (effects (font (size 1.27 1.27)) (justify left bottom))
   )
